Commit message: added a joint to a wheel link

File: robot_description/urdf/robot.urdf (robot description, URDF)
Before this commit: robot robot, 1 links, 0 joints
Links:
- added link link_left_wheel, mass 1; collision cylinder length=0.12 radius=0.08; collision cylinder length=0.12 radius=0.4
Joints:
- added joint joint_chassis_left_wheel: type continuous, parent link_chassis, child link_left_wheel, origin xyz=-0.5 0.65 0 rpy=0 0 0, axis 0 1 0, limit effort=10000 velocity=1000

Commit message: right wheel and hubcaps added

File: robot_description/urdf/robot.urdf (robot description, URDF)
Before this commit: robot robot, 2 links, 1 joints
Links:
- added link link_caster_wheel, mass 1; collision sphere radius=0.10; collision sphere radius=0.2
- added link link_right_wheel, mass 1; collision cylinder length=0.12 radius=0.08; collision cylinder length=0.12 radius=0.4
- link link_left_wheel: geometry collision cylinder length=0.12 radius=0.08; collision cylinder length=0.12 radius=0.4
Joints:
- added joint joint_chassis_caster_wheel: type fixed, parent link_chassis, child link_caster_wheel, origin xyz=0.8 0 -0.15 rpy=0 0 0
- added joint joint_chassis_right_wheel: type continuous, parent link_chassis, child link_right_wheel, origin xyz=-0.5 -0.65 0 rpy=0 0 0, axis 0 1 0, limit effort=10000 velocity=1000

Commit message: exercise 2.3.1 complete: meshes for chassis and wheels included in /meshes, setup.py, and URDF visual elements

File: robot_description/urdf/robot.urdf (robot description, URDF)
Before this commit: robot robot, 4 links, 3 joints
Links:
- link link_chassis: geometry collision box size=2 1.3 0.4; visual mesh filename=package://robot_description/meshes/chassis.stl
- link link_left_wheel: geometry collision cylinder length=0.12 radius=0.08; collision cylinder length=0.12 radius=0.4
- link link_right_wheel: geometry collision cylinder length=0.12 radius=0.08; collision cylinder length=0.12 radius=0.4

Commit message: added laser scan plugin and display_scan node & executable to use laser topic bridge

File: robot_description/urdf/robot.urdf (robot description, URDF)
Before this commit: robot robot, 4 links, 3 joints
Links:
- added link link_laser_scan, mass 0.5; collision cylinder length=0.20 radius=0.15; visual cylinder length=0.20 radius=0.15
Joints:
- added joint joint_laser_scan_chassis: type fixed, parent link_chassis, child link_laser_scan, origin xyz=0.8 0 0.3 rpy=0 0 0
