Commit message: example of splitting URDF into XACRO definition file for links/joints and gazebo file reference containing gazebo tags. modifications to setup.py and launch

File: robot_description/urdf/robot.xacro (robot description, xacro)
@@ -1,78 +1,5 @@
-<?xml version="1.0"?>
-<robot name="robot">
-    <!-- Materials -->
-    <gazebo reference="link_chassis">
-        <visual>
-            <material> <!-- Blue -->
-                <ambient>0.0 0.0 1.0 1.0</ambient>
-                <diffuse>0.0 0.0 1.0 1.0</diffuse>
-                <specular>0.0 0.0 0.0 1.0</specular>
-                <emissive>0.0 0.0 0.0 1.0</emissive>
-            </material>
-        </visual>
-    </gazebo>
-    <gazebo reference="link_caster_wheel">
-        <visual>
-            <material> <!-- Gray -->
-                <ambient>0.25 0.25 0.25 1.0</ambient>
-                <diffuse>0.25 0.25 0.25 1.0</diffuse>
-                <specular>0.0 0.0 0.0 1.0</specular>
-                <emissive>0.0 0.0 0.0 1.0</emissive>
-            </material>
-        </visual>
-        <collision>
-            <surface>
-                <friction>
-                    <ode>
-                        <mu>0.0</mu>
-                        <mu2>0.0</mu2>
-                    </ode>
-                </friction>
-            </surface>
-        </collision>
-    </gazebo>
-    <gazebo reference="link_left_wheel">
-        <visual>
-            <material> <!-- Black -->
-                <ambient>0.1 0.1 0.1 1.0</ambient>
-                <diffuse>0.1 0.1 0.1 1.0</diffuse>
-                <specular>0.0 0.0 0.0 1.0</specular>
-                <emissive>0.0 0.0 0.0 1.0</emissive>
-            </material>
-        </visual>
-        <collision>
-            <surface>
-                <friction>
-                    <ode>
-                        <mu>1.0</mu>
-                        <mu2>1.0</mu2>
-                    </ode>
-                </friction>
-            </surface>
-        </collision>
-    </gazebo>
-    <gazebo reference="link_right_wheel">
-        <visual>
-            <material> <!-- Black -->
-                <ambient>0.1 0.1 0.1 1.0</ambient>
-                <diffuse>0.1 0.1 0.1 1.0</diffuse>
-                <specular>0.0 0.0 0.0 1.0</specular>
-                <emissive>0.0 0.0 0.0 1.0</emissive>
-            </material>
-        </visual>
-        <collision>
-            <surface>
-                <friction>
-                    <ode>
-                        <mu>1.0</mu>
-                        <mu2>1.0</mu2>
-                    </ode>
-                </friction>
-            </surface>
-        </collision>
-    </gazebo>
-    <gazebo reference="joint_chassis_caster_wheel">
-        <preserveFixedJoint>true</preserveFixedJoint>
-    </gazebo>
+<?xml version="1.0" ?>
+<robot name="robot" xmlns:xacro="http://www.ros.org/wiki/xacro">
+    <xacro:include filename="$(find robot_description)/urdf/robot.gazebo" />
     <!-- Link - chassis -->
     <link name="link_chassis">
@@ -261,28 +188,4 @@
         </visual>
     </link>
-    <!-- Differential Drive Plugin -->
-    <gazebo>
-        <plugin
-            filename="libignition-gazebo-diff-drive-system.so"
-            name="ignition::gazebo::systems::DiffDrive">
-            <left_joint>joint_chassis_left_wheel</left_joint>
-            <right_joint>joint_chassis_right_wheel</right_joint>
-            <wheel_separation>1.66</wheel_separation>
-            <wheel_radius>0.4</wheel_radius>
-            <odom_publish_frequency>20</odom_publish_frequency>
-            <topic>cmd_vel</topic>
-            <odom_topic>odom</odom_topic>
-            <tf_topic>tf</tf_topic>
-            <frame_id>odom</frame_id>
-            <child_frame_id>link_chassis</child_frame_id>
-        </plugin>
-    </gazebo>
-    <!-- Gazebo tags - Laser scan -->
-    <gazebo reference="joint_laser_scan_chassis">
-        <preserveFixedJoint>true</preserveFixedJoint>
-    </gazebo>
-    <gazebo reference="link_laser_scan">
-        <material>Gazebo/DarkGrey</material>
-    </gazebo>
     <!-- Laser scan -->
     <joint name="joint_laser_scan_chassis" type="fixed">
@@ -314,55 +217,3 @@
         </collision>
     </link>
-    <!-- Laser Scanner Plugin -->
-    <gazebo>
-        <plugin
-        filename="libignition-gazebo-sensors-system"
-        name="ignition::gazebo::systems::Sensors">
-        <!-- use ogre2 if ogre v2.x is installed, otherwise use ogre -->
-        <render_engine>ogre2</render_engine>
-        </plugin>
-    </gazebo>
-    <gazebo reference="link_laser_scan">
-        <sensor type="gpu_lidar" name="head_hokuyo_sensor">
-            <pose relative_to='lidar_frame'>0 0 0 0 0 0</pose>
-            <always_on>1</always_on>
-            <visualize>true</visualize>
-            <update_rate>20</update_rate>
-            <topic>/laser/scan</topic>
-            <ray>
-                <scan>
-                    <horizontal>
-                        <samples>720</samples>
-                        <resolution>1</resolution>
-                        <min_angle>-1.570796</min_angle>
-                        <max_angle>1.570796</max_angle>
-                    </horizontal>
-                </scan>
-                <range>
-                    <min>0.20</min>
-                    <max>10.0</max>
-                    <resolution>0.01</resolution>
-                </range>
-                <noise>
-                    <type>gaussian</type>
-                    <mean>0.0</mean>
-                    <stddev>0.01</stddev>
-                </noise>
-            </ray>
-        </sensor>
-    </gazebo>
-    <!-- IMU Plugin -->
-    <gazebo>
-        <plugin filename="libignition-gazebo-imu-system"
-            name="ignition::gazebo::systems::Imu">
-        </plugin>
-    </gazebo>
-    <gazebo reference="link_chassis">
-        <sensor name="imu_sensor" type="imu">
-            <always_on>1</always_on>
-            <update_rate>20</update_rate>
-            <visualize>true</visualize>
-            <topic>imu</topic>
-        </sensor>
-    </gazebo>
 </robot>

Commit message: use of parameters and mathematical expressions (of pi) included in xacro

File: robot_description/urdf/robot.xacro (robot description, xacro)
@@ -2,4 +2,7 @@
 <robot name="robot" xmlns:xacro="http://www.ros.org/wiki/xacro">
     <xacro:include filename="$(find robot_description)/urdf/robot.gazebo" />
+    <!-- Parameters -->
+    <xacro:property name="chassis_mass" value="10" />
+    <!--mass value="${1/2 * chassis_mass}" /-->
     <!-- Link - chassis -->
     <link name="link_chassis">
@@ -88,5 +91,5 @@
         <!-- Tires -->
         <collision>
-            <origin rpy="1.5707 0 0" xyz="0 0.18 0" />
+            <origin rpy="${pi/2} 0 0" xyz="0 0.18 0" />
             <geometry>
                 <cylinder length="0.12" radius="0.4"/>
@@ -94,5 +97,5 @@
         </collision>
         <visual>
-            <origin rpy="1.5707 0 0" xyz="0 0.18 0" />
+            <origin rpy="${pi/2} 0 0" xyz="0 0.18 0" />
            <geometry>
                 <mesh filename="package://robot_description/meshes/wheel.stl" />
@@ -104,11 +107,11 @@
         <!-- Axle -->
         <collision>
-            <origin rpy="1.5707 0 0" xyz="0 0.06 0" />
-            <geometry>
-                <cylinder length="0.12" radius="0.08"/>
-            </geometry>
-        </collision>
-        <visual>
-            <origin rpy="1.5707 0 0" xyz="0 0.06 0" />
+            <origin rpy="${pi/2} 0 0" xyz="0 0.06 0" />
+            <geometry>
+                <cylinder length="0.12" radius="0.08"/>
+            </geometry>
+        </collision>
+        <visual>
+            <origin rpy="${pi/2} 0 0" xyz="0 0.06 0" />
             <geometry>
                 <cylinder length="0.12" radius="0.08"/>
@@ -120,5 +123,5 @@
         <!-- Hubcap -->
         <visual>
-            <origin rpy="1.5707 0 0" xyz="0 0.25 0" />
+            <origin rpy="${pi/2} 0 0" xyz="0 0.25 0" />
             <geometry>
                 <box size="0.02 0.5 0.02" />
@@ -147,5 +150,5 @@
         <!-- Tires -->
         <collision>
-            <origin rpy="1.5707 0 0" xyz="0 -0.18 0" />
+            <origin rpy="${pi/2} 0 0" xyz="0 -0.18 0" />
             <geometry>
                 <cylinder length="0.12" radius="0.4"/>
@@ -153,5 +156,5 @@
         </collision>
         <visual>
-            <origin rpy="1.5707 0 0" xyz="0 -0.18 0" />
+            <origin rpy="${pi/2} 0 0" xyz="0 -0.18 0" />
             <geometry>
                 <mesh filename="package://robot_description/meshes/wheel.stl" />
@@ -163,11 +166,11 @@
         <!-- Axle -->
         <collision>
-            <origin rpy="1.5707 0 0" xyz="0 -0.06 0" />
-            <geometry>
-                <cylinder length="0.12" radius="0.08"/>
-            </geometry>
-        </collision>
-        <visual>
-            <origin rpy="1.5707 0 0" xyz="0 -0.06 0" />
+            <origin rpy="${pi/2} 0 0" xyz="0 -0.06 0" />
+            <geometry>
+                <cylinder length="0.12" radius="0.08"/>
+            </geometry>
+        </collision>
+        <visual>
+            <origin rpy="${pi/2} 0 0" xyz="0 -0.06 0" />
             <geometry>
                 <cylinder length="0.12" radius="0.08"/>
@@ -179,5 +182,5 @@
         <!-- Hubcap -->
         <visual>
-            <origin rpy="1.5707 0 0" xyz="0 -0.25 0" />
+            <origin rpy="${pi/2} 0 0" xyz="0 -0.25 0" />
             <geometry>
                 <box size="0.02 0.5 0.02" />
